File: eagle/parametric_eq.sch (EAGLE design)
At the start: 11 parts, among them IC1 TL072P, IC2 TL072P

Commit message: adding components
Parts:
- added C4: 39n, rcl:C-US025-030X050
- added C5: 100n, rcl:C-US025-030X050
- added C6: 5n6, rcl:C-US025-030X050
- added C7: 15n, rcl:C-US025-030X050
- added C8: 1n8, rcl:C-US025-030X050
- added C9: 4n7, rcl:C-US025-030X050
- added R10: 2k2, rcl:R-US_0207/10
- added R11: 1k lin, pot:3RP/1610N
- added R12: 4k7, rcl:R-US_0207/10
- added R13: 5k1, rcl:R-US_0207/10
- added R14, R15: 2k7, rcl:R-US_0207/10
- added R5, R8, R9: 5k lin, pot:3RP/1610N
- R2, R3, R4: value (none) -> 50k log
Connections:
- new net N$1: IC1A.-IN, R10.1
- new net N$2: R10.2, R11.E
Other:
- moved on the sheet: IC1A, R2/2, R4/2
Changed lines of the file:
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@@
 <part name="IC1" library="linear" deviceset="TL072" device="P"/>
 <part name="IC2" library="linear" deviceset="TL072" device="P"/>
-<part name="R2" library="pot" deviceset="3RP/1610G" device=""/>
-<part name="R3" library="pot" deviceset="3RP/1610G" device=""/>
-<part name="R4" library="pot" deviceset="3RP/1610G" device=""/>
+<part name="R2" library="pot" deviceset="3RP/1610G" device="" value="50k log"/>
 <part name="C1" library="rcl" deviceset="C-US" device="025-030X050" value="330p"/>
 <part name="C2" library="rcl" deviceset="C-US" device="025-030X050" value="330p"/>
@@
 <part name="R6" library="rcl" deviceset="R-US_" device="0207/10" value="2k2"/>
 <part name="R7" library="rcl" deviceset="R-US_" device="0207/10" value="2k2"/>
+<part name="R3" library="pot" deviceset="3RP/1610G" device="" value="50k log"/>
+<part name="R4" library="pot" deviceset="3RP/1610G" device="" value="50k log"/>
+<part name="R5" library="pot" deviceset="3RP/1610N" device="" value="5k lin"/>
+<part name="R8" library="pot" deviceset="3RP/1610N" device="" value="5k lin"/>
+<part name="R9" library="pot" deviceset="3RP/1610N" device="" value="5k lin"/>
+<part name="R10" library="rcl" deviceset="R-US_" device="0207/10" value="2k2"/>
+<part name="R11" library="pot" deviceset="3RP/1610N" device="" value="1k lin"/>
+<part name="C4" library="rcl" deviceset="C-US" device="025-030X050" value="39n"/>
+<part name="C5" library="rcl" deviceset="C-US" device="025-030X050" value="100n"/>
+<part name="C6" library="rcl" deviceset="C-US" device="025-030X050" value="5n6"/>
+<part name="C7" library="rcl" deviceset="C-US" device="025-030X050" value="15n"/>
+<part name="C8" library="rcl" deviceset="C-US" device="025-030X050" value="1n8"/>
+<part name="C9" library="rcl" deviceset="C-US" device="025-030X050" value="4n7"/>
+<part name="R12" library="rcl" deviceset="R-US_" device="0207/10" value="4k7"/>
+<part name="R13" library="rcl" deviceset="R-US_" device="0207/10" value="5k1"/>
+<part name="R14" library="rcl" deviceset="R-US_" device="0207/10" value="2k7"/>
+<part name="R15" library="rcl" deviceset="R-US_" device="0207/10" value="2k7"/>
 </parts>
 <sheets>
@@
 </plain>
 <instances>
-<instance part="IC1" gate="A" x="12.7" y="48.26"/>
+<instance part="IC1" gate="A" x="5.08" y="48.26" rot="MR180"/>
 <instance part="IC1" gate="B" x="66.04" y="48.26" rot="MR180"/>
 <instance part="IC2" gate="A" x="111.76" y="48.26" rot="MR180"/>
 <instance part="IC2" gate="B" x="152.4" y="48.26" rot="MR180"/>
 <instance part="R2" gate="/1" x="38.1" y="25.4" rot="MR180"/>
-<instance part="R2" gate="/2" x="53.34" y="25.4" rot="MR180"/>
-<instance part="R3" gate="/1" x="81.28" y="25.4" rot="MR180"/>
-<instance part="R3" gate="/2" x="96.52" y="25.4" rot="MR180"/>
-<instance part="R4" gate="/1" x="127" y="25.4" rot="MR180"/>
-<instance part="R4" gate="/2" x="142.24" y="25.4" rot="MR180"/>
 <instance part="IC1" gate="P" x="-20.32" y="78.74"/>
 <instance part="IC2" gate="P" x="-12.7" y="78.74"/>
@@
 <instance part="R6" gate="G$1" x="111.76" y="73.66"/>
 <instance part="R7" gate="G$1" x="152.4" y="73.66"/>
+<instance part="R2" gate="/2" x="50.8" y="25.4" rot="MR180"/>
+<instance part="R3" gate="/1" x="81.28" y="25.4" rot="MR180"/>
+<instance part="R3" gate="/2" x="96.52" y="25.4" rot="MR180"/>
+<instance part="R4" gate="/1" x="127" y="25.4" rot="MR180"/>
+<instance part="R4" gate="/2" x="139.7" y="25.4" rot="MR180"/>
+<instance part="R5" gate="G$1" x="50.8" y="-10.16" rot="MR90"/>
+<instance part="R8" gate="G$1" x="96.52" y="-10.16" rot="MR90"/>
+<instance part="R9" gate="G$1" x="139.7" y="-10.16" rot="MR90"/>
+<instance part="R10" gate="G$1" x="0" y="66.04"/>
+<instance part="R11" gate="G$1" x="15.24" y="66.04" rot="MR270"/>
+<instance part="C4" gate="G$1" x="25.4" y="22.86" rot="R180"/>
+<instance part="C5" gate="G$1" x="50.8" y="0" rot="R180"/>
+<instance part="C6" gate="G$1" x="68.58" y="22.86" rot="R180"/>
+<instance part="C7" gate="G$1" x="96.52" y="0" rot="R180"/>
+<instance part="C8" gate="G$1" x="114.3" y="22.86" rot="R180"/>
+<instance part="C9" gate="G$1" x="139.7" y="0" rot="R180"/>
+<instance part="R12" gate="G$1" x="50.8" y="12.7" rot="R90"/>
+<instance part="R13" gate="G$1" x="38.1" y="12.7" rot="R90"/>
+<instance part="R14" gate="G$1" x="81.28" y="12.7" rot="R90"/>
+<instance part="R15" gate="G$1" x="96.52" y="12.7" rot="R90"/>
 </instances>
 <busses>
 </busses>
 <nets>
+<net name="N$1" class="0">
+<segment>
+<pinref part="IC1" gate="A" pin="-IN"/>
+<wire x1="-2.54" y1="50.8" x2="-10.16" y2="50.8" width="0.1524" layer="91"/>
+<wire x1="-10.16" y1="50.8" x2="-10.16" y2="66.04" width="0.1524" layer="91"/>
+<pinref part="R10" gate="G$1" pin="1"/>
+<wire x1="-10.16" y1="66.04" x2="-5.08" y2="66.04" width="0.1524" layer="91"/>
+</segment>
+</net>
+<net name="N$2" class="0">
+<segment>
+<pinref part="R10" gate="G$1" pin="2"/>
+<pinref part="R11" gate="G$1" pin="E"/>
+<wire x1="5.08" y1="66.04" x2="10.16" y2="66.04" width="0.1524" layer="91"/>
+</segment>
+</net>
 </nets>
 </sheet>

Commit message: some connections
Parts:
- added R16, R17, R18: 2k2, rcl:R-US_0207/10
- added R19: 4k7, rcl:R-US_0207/10
- added R20: 4k3, rcl:R-US_0207/10
- added U$1: POWER, eurorack:POWER
- R10: value 2k2 -> 5k
- R11: value 1k lin -> 5k
Connections:
- new net +12V: IC1P.V+, IC2P.V+, U$1.+12V
- new net -12V: IC1P.V-, IC2P.V-, U$1.-12V
- new net GND: U$1.GND
- new net N$10: R13.2, R2/1.E
- new net N$11: C5.2, R12.1
- new net N$12: R12.2, R2/2.E
- new net N$13: C5.1, R5.S
- new net N$14: C7.1, R8.S
- new net N$15: C7.2, R15.1
- new net N$16: R15.2, R3/2.E
- new net N$17: R14.2, R3/1.E
- new net N$18: R19.2, R4/1.E
- new net N$19: R20.2, R4/2.E
- new net N$20: C9.2, R20.1
- new net N$21: C9.1, R9.S
- new net N$22: C4.2, IC1B.+IN, R2/1.A, R2/2.A
- new net N$25: R5.E, R8.A
- new net N$26: R8.E, R9.A
- new net N$3: C2.1, IC2A.-IN, R17.2, R6.1
- new net N$4: C3.1, IC2B.-IN, R18.2, R7.1
- new net N$5: C1.1, IC1B.-IN, R1.1, R16.2
- new net N$6: C1.2, IC1B.OUT, R1.2, R17.1
- new net N$7: C2.2, IC2A.OUT, R18.1, R6.2
- new net N$8: C3.2, IC2B.OUT, R7.2
- new net N$9: IC1A.OUT, R11.A, R11.S
Other:
- moved on the sheet: C4, C5, C6, C7, C8, C9, R12, R13, R14, R15, R2/1, R2/2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

Commit message: all components
Parts:
- added C10, C11, C12, C13: 0.1u, rcl:C-US025-030X050
- added LOW: 50k log, pot:3RP/1610G
- R10: value 5k -> 1k
- R2: value 50k log -> 2k; device pot:3RP/1610G -> rcl:R-US_0207/10
- renumbered R3 to MID, R4 to HI
Connections:
- removed net N$25: R5.E, R8.A
- removed net N$26: R8.E, R9.A
- removed net N$9: IC1A.OUT, R11.A, R11.S
- new net N$23: IC1A.OUT, R11.A, R11.S, R16.1, R5.A
- new net N$27: C6.2, IC2A.+IN, MID/1.A, MID/1.S, MID/2.A, MID/2.S
- new net N$28: C8.2, HI/1.A, HI/1.S, HI/2.A, HI/2.S, IC2B.+IN
- net +12V: now also C12.1, C13.1
- net -12V: now also C10.2, C11.2
- net GND: now also C10.1, C11.1, C12.2, C13.2, C4.1, C6.1, C8.1, IC1A.+IN, R13.1, R14.1, R19.1
- net N$1: now also R2.2
- net N$10: now also LOW/1.E; no longer R2/1.E
- net N$12: now also LOW/2.E; no longer R2/2.E
- net N$22: now also LOW/1.A, LOW/1.S, LOW/2.A, LOW/2.S; no longer R2/1.A, R2/2.A
- net N$6: now also R5.E, R8.A
- net N$7: now also R8.E, R9.A
- net N$8: now also R9.E
Other:
- moved on the sheet: IC1A, R10, R11, R16, R17, R18, U$1

Commit message: schematic screenshot
Parts:
- added OUT, OUT1: AUDIO-JACK, erthenvar:AUDIO-JACK
- renumbered R11 to GAIN
Connections:
- new net N$9: OUT1.TIP, R2.1
- net GND: now also OUT.RING, OUT1.RING
- net N$8: now also OUT.TIP
Other:
- moved on the sheet: R2
Changed lines of the file:
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@@
 <layer number="54" name="bGND_GNDA" color="1" fill="9" visible="no" active="no"/>
 <layer number="56" name="wert" color="7" fill="1" visible="no" active="no"/>
+<layer number="57" name="tCAD" color="7" fill="1" visible="no" active="no"/>
 <layer number="90" name="Modules" color="5" fill="1" visible="yes" active="yes"/>
 <layer number="91" name="Nets" color="2" fill="1" visible="yes" active="yes"/>
@@
 <layer number="97" name="Info" color="7" fill="1" visible="yes" active="yes"/>
 <layer number="98" name="Guide" color="6" fill="1" visible="yes" active="yes"/>
+<layer number="99" name="SpiceOrder" color="7" fill="1" visible="yes" active="yes"/>
 <layer number="100" name="Muster" color="7" fill="1" visible="no" active="no"/>
 <layer number="101" name="Patch_Top" color="12" fill="4" visible="yes" active="yes"/>
@@
 <layer number="106" name="bPlate" color="7" fill="1" visible="yes" active="yes"/>
 <layer number="107" name="Crop" color="7" fill="1" visible="yes" active="yes"/>
+<layer number="108" name="tplace-old" color="10" fill="1" visible="yes" active="yes"/>
+<layer number="109" name="ref-old" color="11" fill="1" visible="yes" active="yes"/>
+<layer number="110" name="fp0" color="7" fill="1" visible="yes" active="yes"/>
+<layer number="111" name="LPC17xx" color="7" fill="1" visible="yes" active="yes"/>
+<layer number="112" name="tSilk" color="7" fill="1" visible="yes" active="yes"/>
+<layer number="113" name="IDFDebug" color="4" fill="1" visible="yes" active="yes"/>
 <layer number="116" name="Patch_BOT" color="9" fill="4" visible="yes" active="yes"/>
 <layer number="121" name="_tsilk" color="7" fill="1" visible="yes" active="yes"/>
 <layer number="122" name="_bsilk" color="7" fill="1" visible="yes" active="yes"/>
+<layer number="123" name="tTestmark" color="7" fill="1" visible="yes" active="yes"/>
+<layer number="124" name="bTestmark" color="7" fill="1" visible="yes" active="yes"/>
 <layer number="125" name="_tNames" color="7" fill="1" visible="yes" active="yes"/>
+<layer number="126" name="_bNames" color="7" fill="1" visible="yes" active="yes"/>
+<layer number="127" name="_tValues" color="7" fill="1" visible="yes" active="yes"/>
+<layer number="128" name="_bValues" color="7" fill="1" visible="yes" active="yes"/>
+<layer number="131" name="tAdjust" color="7" fill="1" visible="yes" active="yes"/>
+<layer number="132" name="bAdjust" color="7" fill="1" visible="yes" active="yes"/>
 <layer number="144" name="Drill_legend" color="7" fill="1" visible="yes" active="yes"/>
+<layer number="150" name="Notes" color="7" fill="1" visible="yes" active="yes"/>
 <layer number="151" name="HeatSink" color="7" fill="1" visible="yes" active="yes"/>
+<layer number="152" name="_bDocu" color="7" fill="1" visible="yes" active="yes"/>
+<layer number="153" name="FabDoc1" color="7" fill="1" visible="yes" active="yes"/>
+<layer number="154" name="FabDoc2" color="7" fill="1" visible="yes" active="yes"/>
+<layer number="155" name="FabDoc3" color="7" fill="1" visible="yes" active="yes"/>
+<layer number="199" name="Contour" color="7" fill="1" visible="yes" active="yes"/>
 <layer number="200" name="200bmp" color="1" fill="10" visible="yes" active="yes"/>
 <layer number="201" name="201bmp" color="2" fill="10" visible="yes" active="yes"/>
@@
 <layer number="223" name="223bmp" color="24" fill="1" visible="no" active="no"/>
 <layer number="224" name="224bmp" color="25" fill="1" visible="no" active="no"/>
+<layer number="248" name="Housing" color="7" fill="1" visible="yes" active="yes"/>
+<layer number="249" name="Edge" color="7" fill="1" visible="yes" active="yes"/>
 <layer number="250" name="Descript" color="3" fill="1" visible="no" active="no"/>
 <layer number="251" name="SMDround" color="12" fill="11" visible="no" active="no"/>
@@
 <part name="R9" library="pot" deviceset="3RP/1610N" device="" value="5k lin"/>
 <part name="R10" library="rcl" deviceset="R-US_" device="0207/10" value="1k"/>
-<part name="R11" library="pot" deviceset="3RP/1610N" device="" value="5k"/>
+<part name="GAIN" library="pot" deviceset="3RP/1610N" device="" value="5k"/>
 <part name="C4" library="rcl" deviceset="C-US" device="025-030X050" value="39n"/>
 <part name="C5" library="rcl" deviceset="C-US" device="025-030X050" value="100n"/>
@@
 <part name="C13" library="rcl" deviceset="C-US" device="025-030X050" value="0.1u"/>
 <part name="GND6" library="supply1" deviceset="GND" device=""/>
+<part name="OUT" library="erthenvar" deviceset="AUDIO-JACK" device=""/>
+<part name="GND12" library="supply1" deviceset="GND" device=""/>
+<part name="OUT1" library="erthenvar" deviceset="AUDIO-JACK" device=""/>
+<part name="GND7" library="supply1" deviceset="GND" device=""/>
 </parts>
 <sheets>
@@
 <instance part="R9" gate="G$1" x="160.02" y="-5.08" rot="MR90"/>
 <instance part="R10" gate="G$1" x="27.94" y="91.44"/>
-<instance part="R11" gate="G$1" x="40.64" y="91.44" rot="MR270"/>
+<instance part="GAIN" gate="G$1" x="40.64" y="91.44" rot="MR270"/>
 <instance part="C4" gate="G$1" x="48.26" y="15.24" rot="R180"/>
 <instance part="C5" gate="G$1" x="71.12" y="5.08" rot="R180"/>
@@
 <instance part="GND4" gate="1" x="101.6" y="2.54"/>
 <instance part="GND5" gate="1" x="147.32" y="2.54"/>
-<instance part="R2" gate="G$1" x="10.16" y="76.2"/>
+<instance part="R2" gate="G$1" x="12.7" y="76.2"/>
 <instance part="C10" gate="G$1" x="2.54" y="5.08"/>
 <instance part="C11" gate="G$1" x="27.94" y="5.08"/>
@@
 <instance part="C13" gate="G$1" x="2.54" y="17.78"/>
 <instance part="GND6" gate="1" x="-2.54" y="-7.62"/>
+<instance part="OUT" gate="G$1" x="182.88" y="43.18" rot="R180"/>
+<instance part="GND12" gate="1" x="175.26" y="33.02"/>
+<instance part="OUT1" gate="G$1" x="-5.08" y="71.12" rot="MR180"/>
+<instance part="GND7" gate="1" x="2.54" y="63.5"/>
 </instances>
 <busses>
@@
 <wire x1="20.32" y1="91.44" x2="22.86" y2="91.44" width="0.1524" layer="91"/>
 <pinref part="R2" gate="G$1" pin="2"/>
-<wire x1="15.24" y1="76.2" x2="20.32" y2="76.2" width="0.1524" layer="91"/>
+<wire x1="17.78" y1="76.2" x2="20.32" y2="76.2" width="0.1524" layer="91"/>
 <junction x="20.32" y="76.2"/>
 </segment>
@@
 <segment>
 <pinref part="R10" gate="G$1" pin="2"/>
-<pinref part="R11" gate="G$1" pin="E"/>
+<pinref part="GAIN" gate="G$1" pin="E"/>
 <wire x1="33.02" y1="91.44" x2="35.56" y2="91.44" width="0.1524" layer="91"/>
 </segment>
@@
 <wire x1="175.26" y1="48.26" x2="170.18" y2="48.26" width="0.1524" layer="91"/>
 <junction x="170.18" y="48.26"/>
+<pinref part="OUT" gate="G$1" pin="TIP"/>
 </segment>
 </net>
@@
 <junction x="2.54" y="10.16"/>
 <wire x1="2.54" y1="10.16" x2="2.54" y2="7.62" width="0.1524" layer="91"/>
+</segment>
+<segment>
+<pinref part="OUT" gate="G$1" pin="RING"/>
+<pinref part="GND12" gate="1" pin="GND"/>
+<wire x1="175.26" y1="40.64" x2="175.26" y2="35.56" width="0.1524" layer="91"/>
+</segment>
+<segment>
+<pinref part="OUT1" gate="G$1" pin="RING"/>
+<pinref part="GND7" gate="1" pin="GND"/>
+<wire x1="2.54" y1="66.04" x2="2.54" y2="68.58" width="0.1524" layer="91"/>
 </segment>
 </net>
@@
 <wire x1="38.1" y1="50.8" x2="38.1" y2="63.5" width="0.1524" layer="91"/>
 <junction x="38.1" y="50.8"/>
-<pinref part="R11" gate="G$1" pin="A"/>
+<pinref part="GAIN" gate="G$1" pin="A"/>
 <wire x1="48.26" y1="91.44" x2="45.72" y2="91.44" width="0.1524" layer="91"/>
 <wire x1="48.26" y1="86.36" x2="48.26" y2="91.44" width="0.1524" layer="91"/>
-<pinref part="R11" gate="G$1" pin="S"/>
+<pinref part="GAIN" gate="G$1" pin="S"/>
 <wire x1="40.64" y1="86.36" x2="48.26" y2="86.36" width="0.1524" layer="91"/>
 <junction x="48.26" y="86.36"/>
@@
 </segment>
 </net>
+<net name="N$9" class="0">
+<segment>
+<pinref part="R2" gate="G$1" pin="1"/>
+<pinref part="OUT1" gate="G$1" pin="TIP"/>
+<wire x1="2.54" y1="76.2" x2="7.62" y2="76.2" width="0.1524" layer="91"/>
+</segment>
+</net>

Commit message: bourns ptd pots
Parts:
- removed R5, R8, R9: 5k lin, pot:3RP/1610N
- added LEVEL, LEVEL1, LEVEL2: 5k lin, bourns_ptd:PTD901
- HI, LOW, MID: device pot:3RP/1610G -> bourns_ptd:PTD902PTD902
- renumbered OUT1 to INPUT
Connections:
- net N$13: now also LEVEL.S; no longer R5.S
- net N$14: now also LEVEL1.S; no longer R8.S
- net N$21: now also LEVEL2.S; no longer R9.S
- net N$23: now also LEVEL.A; no longer R5.A
- net N$6: now also LEVEL.E, LEVEL1.A; no longer R5.E, R8.A
- net N$7: now also LEVEL1.E, LEVEL2.A; no longer R8.E, R9.A
- net N$8: now also LEVEL2.E; no longer R9.E

Commit message: parts are on the board
Parts:
- GAIN: value 5k -> 5k lin; device pot:3RP/1610N -> bourns_ptd:PTD901
- renumbered LEVEL to LOLEV, LEVEL1 to MIDLEV, LEVEL2 to HILEV
Connections:
- net N$2: now also GAIN.A; no longer GAIN.E
- net N$23: now also GAIN.E; no longer GAIN.A
Changed lines of the file:
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@@
 <part name="R7" library="rcl" deviceset="R-US_" device="0207/10" value="2k2"/>
 <part name="R10" library="rcl" deviceset="R-US_" device="0207/10" value="1k"/>
-<part name="GAIN" library="pot" deviceset="3RP/1610N" device="" value="5k"/>
 <part name="C4" library="rcl" deviceset="C-US" device="025-030X050" value="39n"/>
 <part name="C5" library="rcl" deviceset="C-US" device="025-030X050" value="100n"/>
@@
 <part name="MID" library="bourns_ptd" deviceset="PTD902" device="" technology="PTD902" value="50k log"/>
 <part name="HI" library="bourns_ptd" deviceset="PTD902" device="" technology="PTD902" value="50k log"/>
-<part name="LEVEL" library="bourns_ptd" deviceset="PTD901" device="" value="5k lin"/>
-<part name="LEVEL1" library="bourns_ptd" deviceset="PTD901" device="" value="5k lin"/>
-<part name="LEVEL2" library="bourns_ptd" deviceset="PTD901" device="" value="5k lin"/>
+<part name="LOLEV" library="bourns_ptd" deviceset="PTD901" device="" value="5k lin"/>
+<part name="MIDLEV" library="bourns_ptd" deviceset="PTD901" device="" value="5k lin"/>
+<part name="HILEV" library="bourns_ptd" deviceset="PTD901" device="" value="5k lin"/>
+<part name="GAIN" library="bourns_ptd" deviceset="PTD901" device="" value="5k lin"/>
 </parts>
 <sheets>
@@
 <instance part="R7" gate="G$1" x="152.4" y="73.66"/>
 <instance part="R10" gate="G$1" x="27.94" y="91.44"/>
-<instance part="GAIN" gate="G$1" x="40.64" y="91.44" rot="MR270"/>
 <instance part="C4" gate="G$1" x="48.26" y="15.24" rot="R180"/>
 <instance part="C5" gate="G$1" x="71.12" y="5.08" rot="R180"/>
@@
 <instance part="HI" gate="/1" x="147.32" y="30.48" rot="MR180"/>
 <instance part="HI" gate="/2" x="160.02" y="30.48" rot="MR180"/>
-<instance part="LEVEL" gate="G$1" x="71.12" y="-5.08" rot="MR90"/>
-<instance part="LEVEL1" gate="G$1" x="116.84" y="-5.08" rot="MR90"/>
-<instance part="LEVEL2" gate="G$1" x="160.02" y="-5.08" rot="MR90"/>
+<instance part="LOLEV" gate="G$1" x="71.12" y="-5.08" rot="MR90"/>
+<instance part="MIDLEV" gate="G$1" x="116.84" y="-5.08" rot="MR90"/>
+<instance part="HILEV" gate="G$1" x="160.02" y="-5.08" rot="MR90"/>
+<instance part="GAIN" gate="G$1" x="40.64" y="91.44" rot="R270"/>
 </instances>
 <busses>
@@
 <segment>
 <pinref part="R10" gate="G$1" pin="2"/>
-<pinref part="GAIN" gate="G$1" pin="E"/>
 <wire x1="33.02" y1="91.44" x2="35.56" y2="91.44" width="0.1524" layer="91"/>
+<pinref part="GAIN" gate="G$1" pin="A"/>
 </segment>
 </net>
@@
 <junction x="78.74" y="48.26"/>
 <junction x="83.82" y="-5.08"/>
-<pinref part="LEVEL" gate="G$1" pin="E"/>
-<pinref part="LEVEL1" gate="G$1" pin="A"/>
+<pinref part="LOLEV" gate="G$1" pin="E"/>
+<pinref part="MIDLEV" gate="G$1" pin="A"/>
 </segment>
 </net>
@@
 <junction x="124.46" y="48.26"/>
 <junction x="129.54" y="-5.08"/>
-<pinref part="LEVEL1" gate="G$1" pin="E"/>
-<pinref part="LEVEL2" gate="G$1" pin="A"/>
+<pinref part="MIDLEV" gate="G$1" pin="E"/>
+<pinref part="HILEV" gate="G$1" pin="A"/>
 </segment>
 </net>
@@
 <junction x="170.18" y="48.26"/>
 <pinref part="OUT" gate="G$1" pin="TIP"/>
-<pinref part="LEVEL2" gate="G$1" pin="E"/>
+<pinref part="HILEV" gate="G$1" pin="E"/>
 </segment>
 </net>
@@
 <pinref part="C5" gate="G$1" pin="1"/>
 <wire x1="71.12" y1="0" x2="71.12" y2="2.54" width="0.1524" layer="91"/>
-<pinref part="LEVEL" gate="G$1" pin="S"/>
+<pinref part="LOLEV" gate="G$1" pin="S"/>
 </segment>
 </net>
@@
 <pinref part="C7" gate="G$1" pin="1"/>
 <wire x1="116.84" y1="0" x2="116.84" y2="2.54" width="0.1524" layer="91"/>
-<pinref part="LEVEL1" gate="G$1" pin="S"/>
+<pinref part="MIDLEV" gate="G$1" pin="S"/>
 </segment>
 </net>
@@
 <pinref part="C9" gate="G$1" pin="1"/>
 <wire x1="160.02" y1="2.54" x2="160.02" y2="0" width="0.1524" layer="91"/>
-<pinref part="LEVEL2" gate="G$1" pin="S"/>
+<pinref part="HILEV" gate="G$1" pin="S"/>
 </segment>
 </net>
@@
 <wire x1="38.1" y1="50.8" x2="38.1" y2="63.5" width="0.1524" layer="91"/>
 <junction x="38.1" y="50.8"/>
-<pinref part="GAIN" gate="G$1" pin="A"/>
 <wire x1="48.26" y1="91.44" x2="45.72" y2="91.44" width="0.1524" layer="91"/>
 <wire x1="48.26" y1="86.36" x2="48.26" y2="91.44" width="0.1524" layer="91"/>
-<pinref part="GAIN" gate="G$1" pin="S"/>
 <wire x1="40.64" y1="86.36" x2="48.26" y2="86.36" width="0.1524" layer="91"/>
 <junction x="48.26" y="86.36"/>
@@
 <wire x1="48.26" y1="63.5" x2="48.26" y2="73.66" width="0.1524" layer="91"/>
 <junction x="48.26" y="73.66"/>
-<pinref part="LEVEL" gate="G$1" pin="A"/>
-</segment>
-</net>
+<pinref part="LOLEV" gate="G$1" pin="A"/>
+<pinref part="GAIN" gate="G$1" pin="E"/>
+<pinref part="GAIN" gate="G$1" pin="S"/>
+</segment>
+</net>
